Commit message: add AMR controller

File: env/models/mobile_manipulator.urdf (robot description, URDF)
Before this commit: robot mobile_manipulator, 28 links, 27 joints
Joints:
- joint base_joint: origin xyz=0 0 0.3 rpy=0 0 0 -> xyz=0 0 0.1 rpy=0 0 0

Commit message: add pre-grasp

File: env/models/mobile_manipulator.urdf (robot description, URDF)
Before this commit: robot mobile_manipulator, 28 links, 27 joints
Links:
- link link_chassis: mass 50 -> 200

Commit message: 241117

File: env/models/mobile_manipulator.urdf (robot description, URDF)
Before this commit: robot mobile_manipulator, 28 links, 27 joints
Links:
- added link box; collision box size=0.01 0.59 0.1; collision box size=0.01 0.59 0.1
- link link_chassis: geometry visual mesh filename=package://syntec/meshes/amr_all.stl scale=0.001 0.001 0.001
Joints:
- added joint box—joint: type fixed, parent link_chassis, child box, origin xyz=0 0 0 rpy=0 0 0
- joint base-base_link: origin xyz=0 0 0.38 rpy=1.570795 0 0 -> xyz=0.205 0 0.745 rpy=1.570795 0 3.14
- joint base_joint: origin xyz=0 0 0.1 rpy=0 0 0 -> xyz=0 0 0.1 rpy=0 0 -3.14
