Commit message: 241225

File: sam_ws/src/pybullet_ros/env/models/tm5_900_with_gripper_h.urdf (robot description, URDF)
Before this commit: robot mobile_manipulator, 29 links, 28 joints
Links:
- removed link box
- removed link car_base
- removed link front_left_caster
- removed link front_right_caster
- removed link link_chassis
- removed link link_left_wheel
- removed link link_right_wheel
- removed link rear_left_caster
- removed link rear_right_caster
- added link base
- link arm_1_link: geometry collision mesh filename=package://meshes/collision/tm5_900_arm1_c.stl; visual mesh filename=package://meshes/visual/tm5_900_arm1.obj
- link arm_2_link: geometry collision mesh filename=package://meshes/collision/tm5_900_arm2_c.stl; visual mesh filename=package://meshes/visual/tm5_900_arm2.obj
- link base_link: geometry collision mesh filename=package://meshes/collision/tm5_base_c.stl; visual mesh filename=package://meshes/visual/tm5_base.obj
- link camera_link: geometry collision box size=0.02505 0.09 0.025; visual mesh filename=package://meshes/collision/d435.dae
- link left_inner_finger: geometry collision mesh filename=package://meshes/collision/robotiq_arg2f_85_inner_finger.dae scale=0.001 0.001 0.001; visual mesh filename=package://meshes/visual/robotiq_arg2f_85_inner_finger.dae scale=0.001 0.001 0.001
- link left_inner_finger_pad: mass 1. -> 0.02
- link left_inner_knuckle: geometry collision mesh filename=package://meshes/collision/robotiq_arg2f_85_inner_knuckle.d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 scale=0.001 0.001 0.001; visual mesh filename=package://meshes/visual/robotiq_arg2f_85_inner_knuckle.dae scale=0.001 0.001 0.001
- link left_outer_finger: geometry collision mesh filename=package://meshes/collision/robotiq_arg2f_85_outer_finger.dae scale=0.001 0.001 0.001; visual mesh filename=package://meshes/visual/robotiq_arg2f_85_outer_finger.dae scale=0.001 0.001 0.001
- link left_outer_knuckle: geometry collision mesh filename=package://meshes/collision/robotiq_arg2f_85_outer_knuckle.d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 scale=0.001 0.001 0.001; visual mesh filename=package://meshes/visual/robotiq_arg2f_85_outer_knuckle.dae scale=0.001 0.001 0.001
- link right_inner_finger: geometry collision mesh filename=package://meshes/collision/robotiq_arg2f_85_inner_finger.dae scale=0.001 0.001 0.001; visual mesh filename=package://meshes/visual/robotiq_arg2f_85_inner_finger.dae scale=0.001 0.001 0.001
- link right_inner_finger_pad: mass 1 -> 0.02
- link right_inner_knuckle: geometry collision mesh filename=package://meshes/collision/robotiq_arg2f_85_inner_knuckle.d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 scale=0.001 0.001 0.001; visual mesh filename=package://meshes/visual/robotiq_arg2f_85_inner_knuckle.dae scale=0.001 0.001 0.001
- link right_outer_finger: geometry collision mesh filename=package://meshes/collision/robotiq_arg2f_85_outer_finger.dae scale=0.001 0.001 0.001; visual mesh filename=package://meshes/visual/robotiq_arg2f_85_outer_finger.dae scale=0.001 0.001 0.001
- link right_outer_knuckle: geometry collision mesh filename=package://meshes/collision/robotiq_arg2f_85_outer_knuckle.d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 scale=0.001 0.001 0.001; visual mesh filename=package://meshes/visual/robotiq_arg2f_85_outer_knuckle.dae scale=0.001 0.001 0.001
- link robotiq_arg2f_base_link: geometry collision mesh filename=package://meshes/collision/robotiq_arg2f_base_link.stl; visual mesh filename=package://meshes/visual/robotiq_arg2f_85_base_link.dae scale=0.001 0.001 0.001
- link shoulder_1_link: geometry collision mesh filename=package://meshes/collision/tm_400w_01_c.stl; visual mesh filename=package://meshes/visual/tm_400w_01.obj
- link wrist_1_link: geometry collision mesh filename=package://meshes/collision/tm_100w_01_c.stl; visual mesh filename=package://meshes/visual/tm_100w_01.obj
- link wrist_2_link: geometry collision mesh filename=package://meshes/collision/tm_100w_02_c.stl; visual mesh filename=package://meshes/visual/tm_100w_02.obj
- link wrist_3_link: geometry collision mesh filename=package://meshes/collision/tm_ee_c.stl; visual mesh filename=package://meshes/visual/tm_ee.obj
Joints:
- removed joint base_joint
- removed joint box—joint
- removed joint front_left_caster_joint
- removed joint front_right_caster_joint
- removed joint joint_left_wheel
- removed joint joint_right_wheel
- removed joint rear_left_caster_joint
- removed joint rear_right_caster_joint
- joint base-base_link: origin xyz=0.205 0 0.745 rpy=1.570795 0 3.14 -> xyz=0 0 0 rpy=1.570795 0 0; parent link_chassis -> base
